File: PCB/Solo_MultiCharger.brd (EAGLE design)
At the start: 91.4 x 99.1 mm, 271 parts, among them J2 68021-410HLF, Q1 DMP3017SFG-7, Q10 2N7002P, Q11 DMP3017SFG-7, Q12 2N7002P, Q13 AON6980, Q14 DMP3017SFG-7, Q15 2N7002P, Q16 AON6980, Q17 AON6980, Q2 2N7002P, Q3 AON6980, Q4 DMP3017SFG-7, Q5 2N7002P, Q6 DMP3017SFG-7, Q7 AON6980, Q8 2N7002P, Q9 DMP3017SFG-7, U1 CS30CL, U10 MCP19035-AAABE/MF, U11 MC78M12CDTG, U12 MCP6L01UT-E/OT, U13 MCP6L01UT-E/OT, U14 MC78M05CDTG, U15 CS30CL, U16 MCP6L01UT-E/OT, U2 MCP19035-AAABE/MF, U3 PIC16F1773-I/SS, U4 CS30CL, U5 MCP19035-AAABE/MF, U6 CS30CL, U7 MCP19035-AAABE/MF, U8 MCP19035-AAABE/MF, U9 CS30CL

Commit message: Increase min via drill to 12mil
Routing:
- net +16.8(2)V: track 134.1 -> 142.8 mm
- net GND: track 109.5 -> 106.1 mm, vias 282 -> 293
- net N$7: track 4.46 -> 2.56 mm, vias 13 -> 12
- net N$30: track 16.1 -> 14.9 mm, vias 11 -> 10
- net N$33: track 9.15 -> 8.33 mm, vias 11 -> 10
- net N$14: track 16.4 -> 15.6 mm, vias 11 -> 10
- net N$50: track 4.24 -> 3.91 mm, vias 13 -> 12
- net +24V: vias 48 -> 49

Commit message: A few small layout changes
Parts:
- added TP1, TP2, TP3, TP4, TP5: TESTPAD, dan:TESTPAD
- moved J1 5.11 mm to (3.96, 55.1)
Connections:
- net +16.8(1)V: now also TP1.TP
- net +16.8(2)V: now also TP2.TP
- net 5V_USB1: now also TP3.TP
- net 5V_USB2: now also TP4.TP
- net N$75: now also TP5.TP
Routing:
- net N$21: track 0.00 -> 6.34 mm
- net N$59: track 0.00 -> 2.28 mm
- net N$31: track 3.20 -> 2.43 mm
- net N$16: track 4.36 -> 3.65 mm
- net N$58: track 4.36 -> 3.65 mm
- net N$8: track 4.66 -> 4.00 mm
- net N$51: track 3.20 -> 2.54 mm
- net N$9: track 3.12 -> 2.53 mm
- net N$15: track 3.20 -> 2.69 mm
- net GND: track 106.1 -> 105.9 mm, vias 293 -> 286
Other:
- board text added: "TP1"
- board text added: "TP2"
- board text added: "TP3"
- board text added: "TP4"
- board text added: "TP5"
